File: Squircuit 2024/Squircuit.kicad_pcb (KiCad board)
At the start: 4 copper layers, 153.7 x 95.2 mm, 59 parts, among them J1 Rudder Encoder, J10 Serial Wire Debug, J11 Encoder Power, J12 Orin, J14 UART, J15 Receiver Inner, J16 SPI 0, J18 HV Relay, J2 Winch Encoder, J20 Magnetometer Inner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

Commit message: Added the relay driver module
Parts:
- removed D2: 1N4001, Diode_THT:D_DO-41_SOD81_P10.16mm_Horizontal
- removed JP1: Jumper_2_Open, Connector_PinHeader_2.54mm:PinHeader_1x02_P2.54mm_Vertical
- removed R19: 10K, Resistor_THT:R_Axial_DIN0207_L6.3mm_D2.5mm_P10.16mm_Horizontal
- removed the REF** at (73.7, 17.1)
- added ?: , , F.Cu at (55.4, 80.8)
- added REF**: MountingHole_4mm, MountingHole:MountingHole_4mm, F.Cu at (55.4, 17.3)
- added REF**: MountingHole_4mm, MountingHole:MountingHole_4mm, F.Cu at (55.4, 80.8)
- added U4: L7812, Package_TO_SOT_THT:TO-220-3_Vertical, F.Cu at (21.6, 90.4)
- added U5: L7812, Package_TO_SOT_THT:TO-220-3_Vertical, F.Cu at (21.6, 84.5)
- added U6: L7812, Package_TO_SOT_THT:TO-220-3_Vertical, F.Cu at (21.6, 78.5)
- added U7: L7812, Package_TO_SOT_THT:TO-220-3_Vertical, F.Cu at (21.6, 72.5)
- added U8: L7812, Package_TO_SOT_THT:TO-220-3_Vertical, F.Cu at (21.6, 66.6)
- added U9: L7812, Package_TO_SOT_THT:TO-220-3_Vertical, F.Cu at (21.6, 60.6)
- Q2: value SIHLU024-GE3 -> 2N3904; footprint Package_TO_SOT_THT:TO-251-3-1EP_Horizontal_TabDown -> Package_TO_SOT_THT:TO-92_Inline
- moved Q2 1.64 mm to (47.9, 28.6)
- moved J11 1.26 mm to (26.7, 86.4)
Connections:
- J7 pad 1: +15V -> Net-(J7-Pin_1)
- J7 pad 2: Net-(D2-A) -> GNDREF
- Q2 pad 1: Net-(Q2-G) -> GNDREF
- Q2 pad 2: Net-(D1-A) -> Net-(Q2-B)
- Q2 pad 3: GNDREF -> Net-(D1-A)
- R15 pad 1: Net-(Q2-G) -> Net-(Q2-B)
- R16 pad 2: Net-(Q2-G) -> Net-(Q2-B)
Routing:
- net Net-(J7-Pin_1): track 0.00 -> 42.4 mm
- net +15V: track 220.5 -> 256.8 mm
- net Net-(D2-A): track 35.8 -> 0.00 mm
- net Net-(Q2-B): track 0.00 -> 13.6 mm
- net Net-(Q2-G): track 13.3 -> 0.00 mm
- net /Ch3d: track 44.1 -> 37.7 mm
- net /AGND: track 88.1 -> 94.3 mm
- net +5V: track 102.7 -> 96.6 mm
- net /SCL: track 74.6 -> 80.6 mm
- net /Ch1d: track 31.6 -> 37.6 mm
- net /SDA: track 75.2 -> 77.8 mm
- net /Ch2d: track 37.8 -> 35.7 mm
- net Net-(D1-A): track 34.6 -> 36.4 mm
- net +3.3V: track 271.5 -> 272.2 mm
- net Net-(J1-Pin_1): track 111.4 -> 110.8 mm
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- removed copper zone on B.Cu, net GNDREF
- removed copper zone on F.Cu, net GNDREF
- removed copper zone on In1.Cu, net GNDREF
