File: Squircuit 2024/Squircuit.kicad_sch (KiCad schematic)
At the start: 55 parts, among them J1 Rudder Encoder, J10 Serial Wire Debug, J11 Encoder Power, J12 Orin, J14 UART, J15 Receiver Inner, J16 SPI 0, J18 HV Relay, J2 Winch Encoder, J20 Magnetometer Inner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

Commit message: Added the relay driver module
Parts:
- removed D2: 1N4001, Diode_THT:D_DO-41_SOD81_P10.16mm_Horizontal, symbol Diode:1N4001
- removed JP1: Jumper_2_Open, Connector_PinHeader_2.54mm:PinHeader_1x02_P2.54mm_Vertical, symbol Jumper:Jumper_2_Open
- removed Q2: SIHLU024-GE3, Package_TO_SOT_THT:TO-251-3-1EP_Horizontal_TabDown, symbol Transistor_FET:IRF740
- removed R19: 10K, Resistor_THT:R_Axial_DIN0207_L6.3mm_D2.5mm_P10.16mm_Horizontal, symbol PCM_SL_Devices:Resistor
- added Q2: 2N3904, Package_TO_SOT_THT:TO-92_Inline, symbol Transistor_BJT:2N3904
- added U4, U5, U6, U7, U8, U9: L7812, Package_TO_SOT_THT:TO-220-3_Vertical, symbol Regulator_Linear:L7812
Connections:
- net +15V: now also U4.1 (IN), U5.1 (IN), U6.1 (IN), U7.1 (IN), U8.1 (IN), U9.1 (IN); no longer J7.1 (Pin_1)
- net GNDREF: now also J7.2 (Pin_2), Q2.1 (E), U4.2 (GND), U5.2 (GND), U6.2 (GND), U7.2 (GND), U8.2 (GND), U9.2 (GND)
- net at R15.1, R16.2: now also Q2.2 (B)
- net at D1.2 (A), J18.2 (Pin_2): now also Q2.3 (C)
- new net: J7.1 (Pin_1), U4.3 (OUT), U5.3 (OUT), U6.3 (OUT), U7.3 (OUT), U8.3 (OUT), U9.3 (OUT)
Other:
- moved on the sheet: J7
